File: Motor-Controller-PCB.kicad_pcb (KiCad board)
At the start: 2 copper layers, 68.6 x 53.3 mm, 32 parts, among them Q1 IFX007T, Q2 TJ200F04M3L, Q3 TJ200F04M3L, U1 DS18B20-PAR

Commit message: Update Motor-Controller-PCB.kicad_pcb
Parts:
- added REF**: SolderWire-0.25sqmm_1x03_P4.2mm_D0.65mm_OD1.7mm, Connector_Wire:SolderWire-0.25sqmm_1x03_P4.2mm_D0.65mm_OD1.7mm, F.Cu at (117.2, 91.8)
Routing:
- net Net-(A1-Pad5): track 0.17 -> 50.8 mm
- net Net-(A1-Pad15): track 0.00 -> 22.2 mm
- net Net-(A1-Pad10): track 38.2 -> 36.9 mm

Commit message: giant cubes
giant cubes
Parts:
- removed the REF** at (122.5, 112.8)
- removed the REF** at (177.1, 118.6)
- removed the REF** at (177.5, 80.0)
- removed the REF** at (124.6, 84.1)
- added REF**: GiantMetalCube, Motor-Controller-PCB:GiantMetalCube, B.Cu at (177.8, 72.8)
- added REF**: GiantMetalCube, Motor-Controller-PCB:GiantMetalCube, B.Cu at (177.5, 109.6)
- added REF**: GiantMetalCube, Motor-Controller-PCB:GiantMetalCube, B.Cu at (119.6, 82.7)
- added REF**: GiantMetalCube, Motor-Controller-PCB:GiantMetalCube, B.Cu at (125.4, 103.4)
